Commit message: 座標軸が逆になっていたため修正

File: wormy_arm_description/urdf/wormy_short_macro.urdf.xacro (robot description, xacro)
@@ -198,5 +198,5 @@
         </collision>
         <inertial>
-            <origin xyz="1.15284e-18 5.6599e-06 -0.0118831" rpy="0 0 0" />
+            <origin xyz="1.15295e-18 5.6599e-06 -0.0118831" rpy="0 0 0" />
             <mass value="0.0234539" />
             <inertia ixx="5.31243e-06" ixy="-1.55552e-37" ixz="-2.05025e-10" iyy="5.31245e-06"
@@ -208,5 +208,5 @@
         <parent link="link_5" />
         <child link="joint_connector_a2" />
-        <axis xyz="0 0 1" />
+        <axis xyz="0 0 -1" />
         <limit lower="-${150/180 * pi}" upper="${150/180 * pi}" effort="1000" velocity="3.14"/>
         <joint_properties friction="0.0" />
@@ -216,5 +216,5 @@
         <parent link="link_4" />
         <child link="link_5" />
-        <axis xyz="0 0 1" />
+        <axis xyz="0 0 -1" />
         <limit lower="-${150/180 * pi}" upper="${150/180 * pi}" effort="1000" velocity="3.14"/>
         <joint_properties friction="0.0" />
@@ -224,5 +224,5 @@
         <parent link="link_3" />
         <child link="link_4" />
-        <axis xyz="0 0 1" />
+        <axis xyz="0 0 -1" />
         <limit lower="-${150/180 * pi}" upper="${150/180 * pi}" effort="1000" velocity="3.14"/>
         <joint_properties friction="0.0" />
@@ -232,5 +232,5 @@
         <parent link="link_2" />
         <child link="link_3" />
-        <axis xyz="0 0 1" />
+        <axis xyz="0 0 -1" />
         <limit lower="-${150/180 * pi}" upper="${150/180 * pi}" effort="1000" velocity="3.14"/>
         <joint_properties friction="0.0" />
@@ -240,5 +240,5 @@
         <parent link="link_1" />
         <child link="link_2" />
-        <axis xyz="0 0 1" />
+        <axis xyz="0 0 -1" />
         <limit lower="-${150/180 * pi}" upper="${150/180 * pi}" effort="1000" velocity="3.14"/>
         <joint_properties friction="0.0" />
@@ -248,5 +248,5 @@
         <parent link="link_0" />
         <child link="link_1" />
-        <axis xyz="0 0 1" />
+        <axis xyz="0 0 -1" />
         <limit lower="-${150/180 * pi}" upper="${150/180 * pi}" effort="1000" velocity="3.14"/>
         <joint_properties friction="0.0" />
